Commit message: updated urdf

File: src/robot_model/urdf/model.urdf (robot description, URDF)
Before this commit: robot myfirst, 6 links, 5 joints
Joints:
- joint base_sphere_joint: axis 0 0 0 -> 0 1 1; type fixed -> continuous

Commit message: modified the urdf & added a simple map

File: src/robot_model/urdf/model.urdf (robot description, URDF)
Before this commit: robot myfirst, 6 links, 5 joints
Joints:
- joint base_imu_joint: origin xyz=-0.05 0 0.105 -> xyz=0.05 0 0.105
- joint base_left_wheel_joint: origin xyz=0.1 -0.125 0 -> xyz=-0.1 0.125 0
- joint base_lidar_joint: origin xyz=-0.1 0 0.105 -> xyz=0.1 0 0.105
- joint base_right_wheel_joint: origin xyz=0.1 0.125 0 -> xyz=-0.1 -0.125 0
- joint base_sphere_joint: origin xyz=-0.1 0 0 -> xyz=0.1 0 0
